File: board/rst-pwr.kicad_pcb (KiCad board)
At the start: 2 copper layers, 94 x 12.7 mm, 5 parts, among them J1 PWR, J2 Molex, J3 RST

Commit message: Updates for new KiCad version.
Signed-off-by: Dan Cross <cross@gajendra.net>
Other:
- net class Default removed
